File: Thermo_Probe/Thermo_Probe.kicad_pcb (KiCad board)
At the start: 2 copper layers, 68.6 x 53.3 mm, 24 parts, among them J1 Power, J2 Digital/PWM, J3 Analog, J4 Digital/PWM, J5 GYRO_CONN, J6 Connector Display, J7 CONN_TEMP, SW1 SW_SPST, SW2 SW_SPST, SW3 SW_SPST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

Commit message: yes
Parts:
- removed MH1, MH2, MH3, MH4: MountingHole_3.2mm, Arduino_MountingHole:MountingHole_3.2mm
- moved R2 1.53 mm to (163.2, 65.0)
- moved R5 1.39 mm to (163.2, 78.2)
- moved R1 0.60 mm to (163.2, 52.1)
Routing:
- net +5V: track 184.9 -> 178.2 mm
- net /button_light: track 65.7 -> 68.5 mm
- net /button_lock: track 32.7 -> 31.3 mm
- net /button_cal: track 26.9 -> 27.8 mm
- net /button_on/off: track 31.2 -> 31.9 mm

Commit message: Probe
Parts:
- moved SW3 4.89 mm to (152.6, 74.5)
- moved R3 4.10 mm to (148.6, 73.6)
- moved RV1 3.16 mm to (153.1, 87.8)
- moved SW2 1.98 mm to (152.6, 63.7)
- moved SW1 1.39 mm to (152.4, 53.0)
- moved R4 1.26 mm to (132.2, 69.8)
- moved R5 1.25 mm to (163.2, 79.5)
- moved R2 0.20 mm to (163.2, 65.2)
Routing:
- net /LED_light: track 26.5 -> 20.4 mm
- net +5V: track 178.2 -> 173.0 mm
- net /button_lock: track 31.3 -> 35.8 mm
- net /Temp_sensor: track 5.77 -> 8.98 mm
- net /button_light: track 68.5 -> 65.7 mm
- net /button_unit: track 17.6 -> 15.4 mm
- net /temp_digital: track 8.74 -> 10.6 mm
- net Net-(D1-A): track 8.61 -> 7.99 mm
Other:
- board text added: "Analog Sensor"
- board text added: "Botton Lock"
- board text added: "Calibration"
- board text added: "On/Off"
- board text added: "Unit"
- board text added: "Version #1 Sebastian Posada 2-3-2025"
