File: Thermo_Probe/Thermo_Probe.kicad_pcb (KiCad board)
At the start: 2 copper layers, 68.6 x 53.3 mm, 20 parts, among them J1 Power, J2 Digital/PWM, J3 Analog, J4 Digital/PWM, J5 GYRO_CONN, J6 Connector Display, J7 CONN_TEMP, SW1 SW_SPST, SW2 SW_SPST, SW3 SW_SPST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

Commit message: new
Parts:
- added G***: LOGO, LOGO, F.Cu at (129.4, 89.8)
- moved J6 25.4 mm to (112.2, 52.9), turned to 90 degrees
- moved J5 22.3 mm to (103.7, 93.2), turned to 90 degrees
Connections:
- J2 pad 1: /I2C_SDA -> /I2C_SCL
- J2 pad 2: /I2C_SCL -> /I2C_SDA
Routing:
- net +5V: track 173.0 -> 230.0 mm
- net /I2C_SCL: track 36.2 -> 47.7 mm
- net /I2C_SDA: track 36.2 -> 47.0 mm
