File: Thermo_Probe/Thermo_Probe.kicad_sch (KiCad schematic)
At the start: 20 parts, among them J1 Power, J2 Digital/PWM, J3 Analog, J4 Digital/PWM, J5 GYRO_CONN, J6 Connector Display, J7 CONN_TEMP, SW1 SW_SPST, SW2 SW_SPST, SW3 SW_SPST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

Commit message: Probe
Other:
- moved on the sheet: D1, J5, J6, J7, R1, R2, R3, R4, R5, R6, RV1, SW1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

Commit message: new
Connections:
- net I2C_SCL: now also J2.1 (Pin_1); no longer J2.2 (Pin_2)
- net I2C_SDA: now also J2.2 (Pin_2); no longer J2.1 (Pin_1)
Changed lines of the file:
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@@
 	)
 	(label "I2C_SDA"
-		(at 78.74 26.67 0)
+		(at 78.74 29.21 0)
 		(effects
 			(font
@@
 	)
 	(label "I2C_SCL"
-		(at 78.74 29.21 0)
+		(at 78.74 26.67 0)
 		(effects
 			(font
